Commit message: update gemini camera's urdf

File: orbbec_description/urdf/gemini_335_336.urdf.xacro (robot description, xacro)
@@ -15,5 +15,5 @@
         </inertial>
         <visual>
-            <origin xyz="0 0 0" rpy="0 0 0" />
+            <origin xyz="-25 0 0" rpy="0 0 0" />
             <geometry>
                 <mesh filename="${mesh_path}camera_link.STL" />
@@ -60,5 +60,5 @@
         <axis xyz="0 0 0" />
     </joint>
-    <link name="camera_infra_1_frame">
+    <link name="camera_left_ir_frame">
         <inertial>
             <origin xyz="-0.00158020887627678 -1.52683853303637E-08 -1.4860800305164E-07"
@@ -70,26 +70,26 @@
         </inertial>
         <visual>
-            <origin xyz="0 0 0" rpy="0 0 0" />
-            <geometry>
-                <mesh filename="${mesh_path}camera_infra_1_frame.STL" />
-            </geometry>
-            <material name="">
-                <color rgba="0.501960784313725 0.250980392156863 0.250980392156863 1" />
-            </material>
-        </visual>
-        <collision>
-            <origin xyz="0 0 0" rpy="0 0 0" />
-            <geometry>
-                <mesh filename="${mesh_path}camera_infra_1_frame.STL" />
-            </geometry>
-        </collision>
-    </link>
-    <joint name="camera_infra_1_joint" type="fixed">
+            <origin xyz="-25 0 0" rpy="0 0 0" />
+            <geometry>
+                <mesh filename="${mesh_path}camera_left_ir_frame.STL" />
+            </geometry>
+            <material name="">
+                <color rgba="0.501960784313725 0.250980392156863 0.250980392156863 1" />
+            </material>
+        </visual>
+        <collision>
+            <origin xyz="0 0 0" rpy="0 0 0" />
+            <geometry>
+                <mesh filename="${mesh_path}camera_left_ir_frame.STL" />
+            </geometry>
+        </collision>
+    </link>
+    <joint name="camera_left_ir_joint" type="fixed">
         <origin xyz="0.01587 -0.025 0.0125" rpy="0 0 0" />
         <parent link="camera_bottom_screw_frame" />
-        <child link="camera_infra_1_frame" />
-        <axis xyz="0 0 0" />
-    </joint>
-    <link name="camera_infra_1_optical_frame">
+        <child link="camera_left_ir_frame" />
+        <axis xyz="0 0 0" />
+    </joint>
+    <link name="camera_left_ir_optical_frame">
         <inertial>
             <origin xyz="1.52683853338331E-08 1.48608003051636E-07 -0.00158020887627678" rpy="0 0 0" />
@@ -102,24 +102,24 @@
             <origin xyz="0 0 0" rpy="0 0 0" />
             <geometry>
-                <mesh filename="${mesh_path}camera_infra_1_optical_frame.STL" />
-            </geometry>
-            <material name="">
-                <color rgba="0.501960784313725 0.250980392156863 0.250980392156863 1" />
-            </material>
-        </visual>
-        <collision>
-            <origin xyz="0 0 0" rpy="0 0 0" />
-            <geometry>
-                <mesh filename="${mesh_path}camera_infra_1_optical_frame.STL" />
-            </geometry>
-        </collision>
-    </link>
-    <joint name="camera_infra_1_optical_joint" type="fixed">
+                <mesh filename="${mesh_path}camera_left_ir_optical_frame.STL" />
+            </geometry>
+            <material name="">
+                <color rgba="0.501960784313725 0.250980392156863 0.250980392156863 1" />
+            </material>
+        </visual>
+        <collision>
+            <origin xyz="0 0 0" rpy="0 0 0" />
+            <geometry>
+                <mesh filename="${mesh_path}camera_left_ir_optical_frame.STL" />
+            </geometry>
+        </collision>
+    </link>
+    <joint name="camera_left_ir_optical_joint" type="fixed">
         <origin xyz="0.01587 -0.025 0.0125" rpy="-1.5707963267949 0 -1.5707963267949" />
         <parent link="camera_bottom_screw_frame" />
-        <child link="camera_infra_1_optical_frame" />
-        <axis xyz="0 0 0" />
-    </joint>
-    <link name="camera_infra2_frame">
+        <child link="camera_left_ir_optical_frame" />
+        <axis xyz="0 0 0" />
+    </joint>
+    <link name="camera_right_ir_frame">
         <inertial>
             <origin xyz="-0.00158020887627678 -1.52683853303637E-08 -1.48608003050581E-07"
@@ -133,24 +133,24 @@
             <origin xyz="0 0 0" rpy="0 0 0" />
             <geometry>
-                <mesh filename="${mesh_path}camera_infra2_frame.STL" />
-            </geometry>
-            <material name="">
-                <color rgba="0.501960784313725 0.250980392156863 0.250980392156863 1" />
-            </material>
-        </visual>
-        <collision>
-            <origin xyz="0 0 0" rpy="0 0 0" />
-            <geometry>
-                <mesh filename="${mesh_path}camera_infra2_frame.STL" />
-            </geometry>
-        </collision>
-    </link>
-    <joint name="camera_infra2_joint" type="fixed">
+                <mesh filename="${mesh_path}camera_right_ir_frame.STL" />
+            </geometry>
+            <material name="">
+                <color rgba="0.501960784313725 0.250980392156863 0.250980392156863 1" />
+            </material>
+        </visual>
+        <collision>
+            <origin xyz="0 0 0" rpy="0 0 0" />
+            <geometry>
+                <mesh filename="${mesh_path}camera_right_ir_frame.STL" />
+            </geometry>
+        </collision>
+    </link>
+    <joint name="camera_right_ir_joint" type="fixed">
         <origin xyz="0.01587 0.025 0.0125" rpy="0 0 0" />
         <parent link="camera_bottom_screw_frame" />
-        <child link="camera_infra2_frame" />
-        <axis xyz="0 0 0" />
-    </joint>
-    <link name="camera_infra2_optical_frame">
+        <child link="camera_right_ir_frame" />
+        <axis xyz="0 0 0" />
+    </joint>
+    <link name="camera_right_ir_optical_frame">
         <inertial>
             <origin xyz="1.52683853268942E-08 1.4860800305058E-07 -0.00158020887627678" rpy="0 0 0" />
@@ -163,21 +163,21 @@
             <origin xyz="0 0 0" rpy="0 0 0" />
             <geometry>
-                <mesh filename="${mesh_path}camera_infra2_optical_frame.STL" />
-            </geometry>
-            <material name="">
-                <color rgba="0.501960784313725 0.250980392156863 0.250980392156863 1" />
-            </material>
-        </visual>
-        <collision>
-            <origin xyz="0 0 0" rpy="0 0 0" />
-            <geometry>
-                <mesh filename="${mesh_path}camera_infra2_optical_frame.STL" />
-            </geometry>
-        </collision>
-    </link>
-    <joint name="camera_infra2_optical_joint" type="fixed">
+                <mesh filename="${mesh_path}camera_right_ir_optical_frame.STL" />
+            </geometry>
+            <material name="">
+                <color rgba="0.501960784313725 0.250980392156863 0.250980392156863 1" />
+            </material>
+        </visual>
+        <collision>
+            <origin xyz="0 0 0" rpy="0 0 0" />
+            <geometry>
+                <mesh filename="${mesh_path}camera_right_ir_optical_frame.STL" />
+            </geometry>
+        </collision>
+    </link>
+    <joint name="camera_right_ir_optical_joint" type="fixed">
         <origin xyz="0.01587 0.025 0.0125" rpy="-1.5707963267949 0 -1.5707963267949" />
         <parent link="camera_bottom_screw_frame" />
-        <child link="camera_infra2_optical_frame" />
+        <child link="camera_right_ir_optical_frame" />
         <axis xyz="0 0 0" />
     </joint>

Commit message: Update orbbec_description

File: orbbec_description/urdf/gemini_335_336.urdf.xacro (robot description, xacro)
@@ -15,5 +15,5 @@
         </inertial>
         <visual>
-            <origin xyz="-25 0 0" rpy="0 0 0" />
+            <origin xyz="0 0 0" rpy="0 0 0" />
             <geometry>
                 <mesh filename="${mesh_path}camera_link.STL" />
