Commit message: Add xacro macro for 335Le camera (#3)
* Similar URDF changes as made for 335L camera including simplified
visual mesh
* Adjusted frame names from Orbbec URDF and added optical frames

File: orbbec_description/urdf/gemini335Le_macro.urdf.xacro (robot description, xacro)
@@ -1,6 +1,6 @@
 <?xml version="1.0" encoding="utf-8"?>
 <robot xmlns:xacro="http://ros.org/wiki/xacro">
-<!-- based off of https://github.com/orbbec/OrbbecSDK_ROS2/blob/v2-main/orbbec_description/urdf/gemini335L_336L.urdf.xarco -->
-<xacro:macro name="gemini_335L_336L" params="
+<!-- based off of orbbec_description/urdf/gemini335Le.urdf.xacro -->
+<xacro:macro name="gemini_335Le" params="
     parent
     prefix:='camera'
@@ -20,9 +20,15 @@
     <inertial>
       <origin
-        xyz="0.00288 0.00062 0.01411"
+        xyz="0.01235 -0.0020872 0.013243"
         rpy="0 0 0" />
       <mass
-        value="0.03307" />
-      <inertia ixx="0.00004" ixy="0" ixz="0" iyy="0.000003" iyz="0" izz="0.00004" />
+        value="0.043446" />
+      <inertia
+        ixx="6.3353E-05"
+        ixy="-1.7904E-06"
+        ixz="-8.8334E-08"
+        iyy="8.2334E-06"
+        iyz="3.3581E-07"
+        izz="6.2898E-05" />
     </inertial>
     <visual>
@@ -32,43 +38,84 @@
       <geometry>
         <mesh
-          filename="file://$(find orbbec_description)/meshes/gemini335L_336L/base_link_simplified.stl" />
+          filename="file://$(find orbbec_description)/meshes/gemini335Le/base_link_simplified.stl" />
       </geometry>
-      <material
-        name="">
-        <color rgba="0.792 0.820 0.933 1" />
+      <material name="">
+        <color rgba="0.8 0.8 0.8 1" />
       </material>
     </visual>
     <collision>
-      <origin xyz="0 0 0.015" rpy="0 0 0" />
+      <origin xyz="0.013 0 0.015" rpy="0 0 0" />
       <geometry>
-        <box size="0.03 0.13 0.03"/>
+        <box size="0.055 0.125 0.03"/>
       </geometry>
     </collision>
   </link>
-  <link name="${prefix}_color_screw_frame" />
-  <joint
-    name="${prefix}_color_screw_frame_joint"
-    type="fixed">
-    <origin
-      xyz="0 0 0"
-      rpy="0 0 0" />
-    <parent
-      link="${prefix}_link" />
-    <child
-      link="${prefix}_color_screw_frame" />
-    <axis
-      xyz="0 0 0" />
-  </joint>
-  <link name="${prefix}_IMU_frame" />
-  <joint
-    name="${prefix}_IMU_frame_joint"
-    type="fixed">
-    <origin
-      xyz="-0.002535 0.039634 0.013243"
-      rpy="0 0 0" />
-    <parent
-      link="${prefix}_color_screw_frame" />
-    <child
-      link="${prefix}_IMU_frame" />
+  <link name="${prefix}_bottom_screw_frame" />
+  <joint
+    name="${prefix}_bottom_screw_frame_joint"
+    type="fixed">
+    <origin
+      xyz="0 0 0"
+      rpy="0 0 0" />
+    <parent
+      link="${prefix}_link" />
+    <child
+      link="${prefix}_bottom_screw_frame" />
+    <axis
+      xyz="0 0 0" />
+  </joint>
+  <link name="${prefix}_infra2_frame" />
+  <joint
+    name="${prefix}_infra2_frame_joint"
+    type="fixed">
+    <origin
+      xyz="0.034005 -0.0475 0.014048"
+      rpy="0 0 0" />
+    <parent
+      link="${prefix}_link" />
+    <child
+      link="${prefix}_infra2_frame" />
+    <axis
+      xyz="0 0 0" />
+  </joint>
+  <link name="${prefix}_infra2_optical_frame" />
+  <joint
+    name="${prefix}_infra2_optical_frame_joint"
+    type="fixed">
+    <origin
+      xyz="0 0 0"
+      rpy="-1.5708 0 -1.5708" />
+    <parent
+      link="${prefix}_infra2_frame" />
+    <child
+      link="${prefix}_infra2_optical_frame" />
+    <axis
+      xyz="0 0 0" />
+  </joint>
+  <link name="${prefix}_infra1_frame" />
+  <joint
+    name="${prefix}_infra1_frame_joint"
+    type="fixed">
+    <origin
+      xyz="0.034005 0.0475 0.014048"
+      rpy="0 0 0" />
+    <parent
+      link="${prefix}_link" />
+    <child
+      link="${prefix}_infra1_frame" />
+    <axis
+      xyz="0 0 0" />
+  </joint>
+  <link name="${prefix}_infra1_optical_frame" />
+  <joint
+    name="${prefix}_infra1_optical_frame_joint"
+    type="fixed">
+    <origin
+      xyz="0 0 0"
+      rpy="-1.5708 0 -1.5708" />
+    <parent
+      link="${prefix}_infra1_frame" />
+    <child
+      link="${prefix}_infra1_optical_frame" />
     <axis
       xyz="0 0 0" />
@@ -78,9 +125,6 @@
     name="${prefix}_depth_frame_joint"
     type="fixed">
-    <origin
-      xyz="0.011715 0.0475 0.014311"
-      rpy="0 0 0" />
-    <parent
-      link="${prefix}_color_screw_frame" />
+    <parent
+      link="${prefix}_infra1_frame" />
     <child
       link="${prefix}_depth_frame" />
@@ -92,95 +136,50 @@
     name="${prefix}_depth_optical_frame_joint"
     type="fixed">
+    <parent
+      link="${prefix}_infra1_optical_frame" />
+    <child
+      link="${prefix}_depth_optical_frame" />
+    <axis
+      xyz="0 0 0" />
+  </joint>
+  <link name="${prefix}_color_frame" />
+  <joint
+    name="${prefix}_frame_frame_joint"
+    type="fixed">
+    <origin
+      xyz="0.034014 0.02375 0.014048"
+      rpy="0 0 0" />
+    <parent
+      link="${prefix}_link" />
+    <child
+      link="${prefix}_color_frame" />
+    <axis
+      xyz="0 0 0" />
+  </joint>
+  <link name="${prefix}_color_optical_frame" />
+  <joint
+    name="${prefix}_color_optical_frame_joint"
+    type="fixed">
     <origin
       xyz="0 0 0"
       rpy="-1.5708 0 -1.5708" />
     <parent
-      link="${prefix}_depth_frame" />
-    <child
-      link="${prefix}_depth_optical_frame" />
-    <axis
-      xyz="0 0 0" />
-  </joint>
-  <link name="${prefix}_infra1_frame" />
-  <joint
-    name="${prefix}_infra1_frame_joint"
-    type="fixed">
-    <origin
-      xyz="0.011715 0.0475 0.014311"
-      rpy="0 0 0" />
-    <parent
-      link="${prefix}_color_screw_frame" />
-    <child
-      link="${prefix}_infra1_frame" />
-    <axis
-      xyz="0 0 0" />
-  </joint>
-  <link name="${prefix}_infra1_optical_frame" />
-  <joint
-    name="${prefix}_infra1_optical_frame_joint"
-    type="fixed">
-    <origin
-      xyz="0 0 0"
-      rpy="-1.5708 0 -1.5708" />
-    <parent
-      link="${prefix}_infra1_frame" />
-    <child
-      link="${prefix}_infra1_optical_frame" />
-    <axis
-      xyz="0 0 0" />
-  </joint>
-  <link name="${prefix}_infra2_frame" />
-  <joint
-    name="${prefix}_infra2_frame_joint"
-    type="fixed">
-    <origin
-      xyz="0.011715 -0.0475 0.014311"
-      rpy="0 0 0" />
-    <parent
-      link="${prefix}_color_screw_frame" />
-    <child
-      link="${prefix}_infra2_frame" />
-    <axis
-      xyz="0 0 0" />
-  </joint>
-  <link name="${prefix}_infra2_optical_frame" />
-  <joint
-    name="${prefix}_infra2_optical_frame_joint"
-    type="fixed">
-    <origin
-      xyz="0 0 0"
-      rpy="-1.5708 0 -1.5708" />
-    <parent
-      link="${prefix}_infra2_frame" />
-    <child
-      link="${prefix}_infra2_optical_frame" />
-    <axis
-      xyz="0 0 0" />
-  </joint>
-  <link name="${prefix}_color_frame" />
-  <joint
-    name="${prefix}_color_frame_joint"
-    type="fixed">
-    <origin
-      xyz="0.011715 0.02375 0.014311"
-      rpy="0.0010157 0 0" />
-    <parent
-      link="${prefix}_color_screw_frame" />
-    <child
       link="${prefix}_color_frame" />
-    <axis
-      xyz="0 0 0" />
-  </joint>
-  <link name="${prefix}_color_optical_frame" />
-  <joint
-    name="${prefix}_color_optical_frame_joint"
-    type="fixed">
-    <origin
-      xyz="0 0 0"
-      rpy="-1.5708 0 -1.5708" />
-    <parent
-      link="${prefix}_color_frame" />
     <child
       link="${prefix}_color_optical_frame" />
+    <axis
+      xyz="0 0 0" />
+  </joint>
+  <link name="${prefix}_imu_frame" />
+  <joint
+    name="${prefix}_imu_frame_joint"
+    type="fixed">
+    <origin
+      xyz="0.019757 0.03619 0.013358"
+      rpy="0 0 0" />
+    <parent
+      link="${prefix}_link" />
+    <child
+      link="${prefix}_imu_frame" />
     <axis
       xyz="0 0 0" />
@@ -198,5 +197,5 @@
       h_fov="${94 * pi/180}"
       v_fov="${68 * pi/180}"
-      min_depth="0.17"
+      min_depth="0.25"
       max_depth="6.0" />
   </xacro:if>

Commit message: switch prefix to name

File: orbbec_description/urdf/gemini335Le_macro.urdf.xacro (robot description, xacro)
@@ -4,5 +4,5 @@
 <xacro:macro name="gemini_335Le" params="
     parent
-    prefix:='camera'
+    name:='camera'
     *origin
     sim_gazebo:=false
@@ -11,11 +11,11 @@
     gz_image_height:='530'">
   <!-- The original link started with camera_link -->
-  <joint name="${prefix}_gemini_mount_fixed_joint" type="fixed">
+  <joint name="${name}_gemini_mount_fixed_joint" type="fixed">
     <parent link="${parent}" />
-    <child link="${prefix}_link" />
+    <child link="${name}_link" />
     <xacro:insert_block name="origin"/>
   </joint>
   <link
-    name="${prefix}_link">
+    name="${name}_link">
     <inertial>
       <origin
@@ -51,21 +51,21 @@
     </collision>
   </link>
-  <link name="${prefix}_bottom_screw_frame" />
-  <joint
-    name="${prefix}_bottom_screw_frame_joint"
-    type="fixed">
-    <origin
-      xyz="0 0 0"
-      rpy="0 0 0" />
-    <parent
-      link="${prefix}_link" />
-    <child
-      link="${prefix}_bottom_screw_frame" />
-    <axis
-      xyz="0 0 0" />
-  </joint>
-  <link name="${prefix}_infra2_frame" />
-  <joint
-    name="${prefix}_infra2_frame_joint"
+  <link name="${name}_bottom_screw_frame" />
+  <joint
+    name="${name}_bottom_screw_frame_joint"
+    type="fixed">
+    <origin
+      xyz="0 0 0"
+      rpy="0 0 0" />
+    <parent
+      link="${name}_link" />
+    <child
+      link="${name}_bottom_screw_frame" />
+    <axis
+      xyz="0 0 0" />
+  </joint>
+  <link name="${name}_infra2_frame" />
+  <joint
+    name="${name}_infra2_frame_joint"
     type="fixed">
     <origin
@@ -73,13 +73,13 @@
       rpy="0 0 0" />
     <parent
-      link="${prefix}_link" />
-    <child
-      link="${prefix}_infra2_frame" />
-    <axis
-      xyz="0 0 0" />
-  </joint>
-  <link name="${prefix}_infra2_optical_frame" />
-  <joint
-    name="${prefix}_infra2_optical_frame_joint"
+      link="${name}_link" />
+    <child
+      link="${name}_infra2_frame" />
+    <axis
+      xyz="0 0 0" />
+  </joint>
+  <link name="${name}_infra2_optical_frame" />
+  <joint
+    name="${name}_infra2_optical_frame_joint"
     type="fixed">
     <origin
@@ -87,13 +87,13 @@
       rpy="-1.5708 0 -1.5708" />
     <parent
-      link="${prefix}_infra2_frame" />
-    <child
-      link="${prefix}_infra2_optical_frame" />
-    <axis
-      xyz="0 0 0" />
-  </joint>
-  <link name="${prefix}_infra1_frame" />
-  <joint
-    name="${prefix}_infra1_frame_joint"
+      link="${name}_infra2_frame" />
+    <child
+      link="${name}_infra2_optical_frame" />
+    <axis
+      xyz="0 0 0" />
+  </joint>
+  <link name="${name}_infra1_frame" />
+  <joint
+    name="${name}_infra1_frame_joint"
     type="fixed">
     <origin
@@ -101,13 +101,13 @@
       rpy="0 0 0" />
     <parent
-      link="${prefix}_link" />
-    <child
-      link="${prefix}_infra1_frame" />
-    <axis
-      xyz="0 0 0" />
-  </joint>
-  <link name="${prefix}_infra1_optical_frame" />
-  <joint
-    name="${prefix}_infra1_optical_frame_joint"
+      link="${name}_link" />
+    <child
+      link="${name}_infra1_frame" />
+    <axis
+      xyz="0 0 0" />
+  </joint>
+  <link name="${name}_infra1_optical_frame" />
+  <joint
+    name="${name}_infra1_optical_frame_joint"
     type="fixed">
     <origin
@@ -115,35 +115,35 @@
       rpy="-1.5708 0 -1.5708" />
     <parent
-      link="${prefix}_infra1_frame" />
-    <child
-      link="${prefix}_infra1_optical_frame" />
-    <axis
-      xyz="0 0 0" />
-  </joint>
-  <link name="${prefix}_depth_frame" />
-  <joint
-    name="${prefix}_depth_frame_joint"
-    type="fixed">
-    <parent
-      link="${prefix}_infra1_frame" />
-    <child
-      link="${prefix}_depth_frame" />
-    <axis
-      xyz="0 0 0" />
-  </joint>
-  <link name="${prefix}_depth_optical_frame" />
-  <joint
-    name="${prefix}_depth_optical_frame_joint"
-    type="fixed">
-    <parent
-      link="${prefix}_infra1_optical_frame" />
-    <child
-      link="${prefix}_depth_optical_frame" />
-    <axis
-      xyz="0 0 0" />
-  </joint>
-  <link name="${prefix}_color_frame" />
-  <joint
-    name="${prefix}_frame_frame_joint"
+      link="${name}_infra1_frame" />
+    <child
+      link="${name}_infra1_optical_frame" />
+    <axis
+      xyz="0 0 0" />
+  </joint>
+  <link name="${name}_depth_frame" />
+  <joint
+    name="${name}_depth_frame_joint"
+    type="fixed">
+    <parent
+      link="${name}_infra1_frame" />
+    <child
+      link="${name}_depth_frame" />
+    <axis
+      xyz="0 0 0" />
+  </joint>
+  <link name="${name}_depth_optical_frame" />
+  <joint
+    name="${name}_depth_optical_frame_joint"
+    type="fixed">
+    <parent
+      link="${name}_infra1_optical_frame" />
+    <child
+      link="${name}_depth_optical_frame" />
+    <axis
+      xyz="0 0 0" />
+  </joint>
+  <link name="${name}_color_frame" />
+  <joint
+    name="${name}_frame_frame_joint"
     type="fixed">
     <origin
@@ -151,13 +151,13 @@
       rpy="0 0 0" />
     <parent
-      link="${prefix}_link" />
-    <child
-      link="${prefix}_color_frame" />
-    <axis
-      xyz="0 0 0" />
-  </joint>
-  <link name="${prefix}_color_optical_frame" />
-  <joint
-    name="${prefix}_color_optical_frame_joint"
+      link="${name}_link" />
+    <child
+      link="${name}_color_frame" />
+    <axis
+      xyz="0 0 0" />
+  </joint>
+  <link name="${name}_color_optical_frame" />
+  <joint
+    name="${name}_color_optical_frame_joint"
     type="fixed">
     <origin
@@ -165,13 +165,13 @@
       rpy="-1.5708 0 -1.5708" />
     <parent
-      link="${prefix}_color_frame" />
-    <child
-      link="${prefix}_color_optical_frame" />
-    <axis
-      xyz="0 0 0" />
-  </joint>
-  <link name="${prefix}_imu_frame" />
-  <joint
-    name="${prefix}_imu_frame_joint"
+      link="${name}_color_frame" />
+    <child
+      link="${name}_color_optical_frame" />
+    <axis
+      xyz="0 0 0" />
+  </joint>
+  <link name="${name}_imu_frame" />
+  <joint
+    name="${name}_imu_frame_joint"
     type="fixed">
     <origin
@@ -179,7 +179,7 @@
       rpy="0 0 0" />
     <parent
-      link="${prefix}_link" />
-    <child
-      link="${prefix}_imu_frame" />
+      link="${name}_link" />
+    <child
+      link="${name}_imu_frame" />
     <axis
       xyz="0 0 0" />
@@ -190,6 +190,6 @@
     <!-- TODO: Upstream changes required for a triggered RBGD camera -->
     <xacro:gazebo_rgbd
-      name="${prefix}"
-      gz_topic_name="${prefix}"
+      name="${name}"
+      gz_topic_name="${name}"
       fps="${gz_fps}"
       image_width="${gz_image_width}"
