Commit message: Remove gz (#8)

File: orbbec_description/urdf/gemini335L_336L_macro.urdf.xacro (robot description, xacro)
@@ -5,9 +5,5 @@
     parent
     prefix:='camera'
-    *origin
-    sim_gazebo:=false
-    gz_fps:='5'
-    gz_image_width:='848'
-    gz_image_height:='530'">
+    *origin">
   <!-- The original link started with camera_link -->
   <joint name="${prefix}_gemini_mount_fixed_joint" type="fixed">
@@ -48,5 +44,5 @@
   <link name="${prefix}_color_screw_frame" />
   <joint
-    name="${prefix}_color_screw_frame_joint"
+    name="${prefix}_color_screw_joint"
     type="fixed">
     <origin
@@ -62,5 +58,5 @@
   <link name="${prefix}_IMU_frame" />
   <joint
-    name="${prefix}_IMU_frame_joint"
+    name="${prefix}_IMU_joint"
     type="fixed">
     <origin
@@ -76,5 +72,5 @@
   <link name="${prefix}_depth_frame" />
   <joint
-    name="${prefix}_depth_frame_joint"
+    name="${prefix}_depth_joint"
     type="fixed">
     <origin
@@ -90,5 +86,5 @@
   <link name="${prefix}_depth_optical_frame" />
   <joint
-    name="${prefix}_depth_optical_frame_joint"
+    name="${prefix}_depth_optical_joint"
     type="fixed">
     <origin
@@ -104,5 +100,5 @@
   <link name="${prefix}_infra1_frame" />
   <joint
-    name="${prefix}_infra1_frame_joint"
+    name="${prefix}_infra1_joint"
     type="fixed">
     <origin
@@ -118,5 +114,5 @@
   <link name="${prefix}_infra1_optical_frame" />
   <joint
-    name="${prefix}_infra1_optical_frame_joint"
+    name="${prefix}_infra1_optical_joint"
     type="fixed">
     <origin
@@ -132,5 +128,5 @@
   <link name="${prefix}_infra2_frame" />
   <joint
-    name="${prefix}_infra2_frame_joint"
+    name="${prefix}_infra2_joint"
     type="fixed">
     <origin
@@ -146,5 +142,5 @@
   <link name="${prefix}_infra2_optical_frame" />
   <joint
-    name="${prefix}_infra2_optical_frame_joint"
+    name="${prefix}_infra2_optical_joint"
     type="fixed">
     <origin
@@ -158,7 +154,15 @@
       xyz="0 0 0" />
   </joint>
-  <link name="${prefix}_color_frame" />
+  <link name="${prefix}_color_frame" >
+    <inertial>
+        <mass value="0.01" />
+        <origin xyz="0 0 0" rpy="0 0 0"/>
+        <inertia ixx="0.001"  ixy="0" ixz="0"
+                 iyx="0" iyy="0.001" iyz="0"
+                 izx="0" izy="0" izz="0.001" />
+      </inertial>
+  </link>
   <joint
-    name="${prefix}_color_frame_joint"
+    name="${prefix}_color_joint"
     type="fixed">
     <origin
@@ -174,5 +178,5 @@
   <link name="${prefix}_color_optical_frame" />
   <joint
-    name="${prefix}_color_optical_frame_joint"
+    name="${prefix}_color_optical_joint"
     type="fixed">
     <origin
@@ -186,19 +190,4 @@
       xyz="0 0 0" />
   </joint>
-  <xacro:if value="${sim_gazebo}">
-    <!-- Use the realsense2_gz_description which can simulate a generic depth camera -->
-    <xacro:include filename="$(find realsense2_gz_description)/urdf/rgbd_camera.gazebo.xacro" />
-    <!-- TODO: Upstream changes required for a triggered RBGD camera -->
-    <xacro:gazebo_rgbd
-      name="${prefix}"
-      gz_topic_name="${prefix}"
-      fps="${gz_fps}"
-      image_width="${gz_image_width}"
-      image_height="${gz_image_height}"
-      h_fov="${94 * pi/180}"
-      v_fov="${68 * pi/180}"
-      min_depth="0.17"
-      max_depth="6.0" />
-  </xacro:if>
 </xacro:macro>
 </robot>

File: orbbec_description/urdf/gemini335Le_macro.urdf.xacro (robot description, xacro)
@@ -5,9 +5,5 @@
     parent
     name:='camera'
-    *origin
-    sim_gazebo:=false
-    gz_fps:='5'
-    gz_image_width:='848'
-    gz_image_height:='530'">
+    *origin">
   <!-- The original link started with camera_link -->
   <joint name="${name}_gemini_mount_fixed_joint" type="fixed">
@@ -53,5 +49,5 @@
   <link name="${name}_bottom_screw_frame" />
   <joint
-    name="${name}_bottom_screw_frame_joint"
+    name="${name}_bottom_screw_joint"
     type="fixed">
     <origin
@@ -67,5 +63,5 @@
   <link name="${name}_infra2_frame" />
   <joint
-    name="${name}_infra2_frame_joint"
+    name="${name}_infra2_joint"
     type="fixed">
     <origin
@@ -81,5 +77,5 @@
   <link name="${name}_infra2_optical_frame" />
   <joint
-    name="${name}_infra2_optical_frame_joint"
+    name="${name}_infra2_optical_joint"
     type="fixed">
     <origin
@@ -95,5 +91,5 @@
   <link name="${name}_infra1_frame" />
   <joint
-    name="${name}_infra1_frame_joint"
+    name="${name}_infra1_joint"
     type="fixed">
     <origin
@@ -109,5 +105,5 @@
   <link name="${name}_infra1_optical_frame" />
   <joint
-    name="${name}_infra1_optical_frame_joint"
+    name="${name}_infra1_optical_joint"
     type="fixed">
     <origin
@@ -123,5 +119,5 @@
   <link name="${name}_depth_frame" />
   <joint
-    name="${name}_depth_frame_joint"
+    name="${name}_depth_joint"
     type="fixed">
     <parent
@@ -134,5 +130,5 @@
   <link name="${name}_depth_optical_frame" />
   <joint
-    name="${name}_depth_optical_frame_joint"
+    name="${name}_depth_optical_joint"
     type="fixed">
     <parent
@@ -143,7 +139,15 @@
       xyz="0 0 0" />
   </joint>
-  <link name="${name}_color_frame" />
+  <link name="${name}_color_frame" >
+    <inertial>
+        <mass value="0.01" />
+        <origin xyz="0 0 0" rpy="0 0 0"/>
+        <inertia ixx="0.001"  ixy="0" ixz="0"
+                 iyx="0" iyy="0.001" iyz="0"
+                 izx="0" izy="0" izz="0.001" />
+      </inertial>
+  </link>
   <joint
-    name="${name}_frame_frame_joint"
+    name="${name}_color_joint"
     type="fixed">
     <origin
@@ -159,5 +163,5 @@
   <link name="${name}_color_optical_frame" />
   <joint
-    name="${name}_color_optical_frame_joint"
+    name="${name}_color_optical_joint"
     type="fixed">
     <origin
@@ -173,5 +177,5 @@
   <link name="${name}_imu_frame" />
   <joint
-    name="${name}_imu_frame_joint"
+    name="${name}_imu_joint"
     type="fixed">
     <origin
@@ -185,19 +189,4 @@
       xyz="0 0 0" />
   </joint>
-  <xacro:if value="${sim_gazebo}">
-    <!-- Use the realsense2_gz_description which can simulate a generic depth camera -->
-    <xacro:include filename="$(find realsense2_gz_description)/urdf/rgbd_camera.gazebo.xacro" />
-    <!-- TODO: Upstream changes required for a triggered RBGD camera -->
-    <xacro:gazebo_rgbd
-      name="${name}"
-      gz_topic_name="${name}"
-      fps="${gz_fps}"
-      image_width="${gz_image_width}"
-      image_height="${gz_image_height}"
-      h_fov="${94 * pi/180}"
-      v_fov="${68 * pi/180}"
-      min_depth="0.25"
-      max_depth="6.0" />
-  </xacro:if>
 </xacro:macro>
 </robot>
