Commit message: Refactor URDF files for camera frames and joints

File: orbbec_description/urdf/gemini335Lg.urdf.xacro (robot description, xacro)
@@ -24,5 +24,5 @@
     <visual>
       <origin
-        xyz="0 0 0"
+        xyz="-0.0117149999999995 -0.0475 -0.0143111800025738"
         rpy="0 0 0" />
       <geometry>
@@ -90,5 +90,5 @@
     type="fixed">
     <origin
-      xyz="0 0 0"
+      xyz="-0.0117149999999995 -0.0475 -0.0143111800025738"
       rpy="0 0 0" />
     <parent
@@ -100,5 +100,5 @@
   </joint>
   <link
-    name="camera_infra1_frame">
+    name="camera_left_ir_frame">
     <inertial>
       <origin
@@ -140,18 +140,18 @@
   </link>
   <joint
-    name="camera_infra1_frame"
-    type="fixed">
-    <origin
-      xyz="0.0117149999999995 0.0475 0.0143111800025738"
+    name="camera_left_ir_frame"
+    type="fixed">
+    <origin
+      xyz="0 0 0"
       rpy="0 0 0" />
     <parent
-      link="camera_bottom_screw_frame" />
-    <child
-      link="camera_infra1_frame" />
-    <axis
-      xyz="0 0 0" />
-  </joint>
-  <link
-    name="camera_infra1_optical_frame">
+      link="camera_depth_frame" />
+    <child
+      link="camera_left_ir_frame" />
+    <axis
+      xyz="0 0 0" />
+  </joint>
+  <link
+    name="camera_left_ir_optical_frame">
     <inertial>
       <origin
@@ -193,5 +193,5 @@
   </link>
   <joint
-    name="camera_infra1_optical_frame"
+    name="camera_left_ir_optical_frame"
     type="fixed">
     <origin
@@ -199,7 +199,7 @@
       rpy="-1.5707963267949 0 -1.5707963267949" />
     <parent
-      link="camera_infra1_frame" />
-    <child
-      link="camera_infra1_optical_frame" />
+      link="camera_left_ir_frame" />
+    <child
+      link="camera_left_ir_optical_frame" />
     <axis
       xyz="0 0 0" />
@@ -249,8 +249,8 @@
     type="fixed">
     <origin
-      xyz="0.0117149999999995 0.02375 0.0143111800025738"
+      xyz="0 -0.023749999701976776 0"
       rpy="0 0 0" />
     <parent
-      link="camera_bottom_screw_frame" />
+      link="camera_depth_frame" />
     <child
       link="camera_color_frame" />
@@ -312,5 +312,5 @@
   </joint>
   <link
-    name="camera_infra2_frame">
+    name="camera_right_ir_frame">
     <inertial>
       <origin
@@ -352,18 +352,18 @@
   </link>
   <joint
-    name="camera_infra2_frame"
-    type="fixed">
-    <origin
-      xyz="0.0117149999999995 -0.0475 0.0143111800025738"
+    name="camera_right_ir_frame"
+    type="fixed">
+    <origin
+      xyz="0 -0.095 0"
       rpy="0 0 0" />
     <parent
-      link="camera_bottom_screw_frame" />
-    <child
-      link="camera_infra2_frame" />
-    <axis
-      xyz="0 0 0" />
-  </joint>
-  <link
-    name="camera_infra2_optical_frame">
+      link="camera_depth_frame" />
+    <child
+      link="camera_right_ir_frame" />
+    <axis
+      xyz="0 0 0" />
+  </joint>
+  <link
+    name="camera_right_ir_optical_frame">
     <inertial>
       <origin
@@ -405,5 +405,5 @@
   </link>
   <joint
-    name="camera_infra2_optical_frame"
+    name="camera_right_ir_optical_frame"
     type="fixed">
     <origin
@@ -411,12 +411,12 @@
       rpy="-1.57079632679486 0 -1.5707963267949" />
     <parent
-      link="camera_infra2_frame" />
-    <child
-      link="camera_infra2_optical_frame" />
-    <axis
-      xyz="0 0 0" />
-  </joint>
-  <link
-    name="camera_IMU_frame">
+      link="camera_right_ir_frame" />
+    <child
+      link="camera_right_ir_optical_frame" />
+    <axis
+      xyz="0 0 0" />
+  </joint>
+  <link
+    name="camera_imu_frame">
     <inertial>
       <origin
@@ -458,13 +458,13 @@
   </link>
   <joint
-    name="camera_IMU_frame"
-    type="fixed">
-    <origin
-      xyz="-0.00253500000000046 0.036187989999999 0.0136240800025733"
+    name="camera_imu_frame"
+    type="fixed">
+    <origin
+      xyz="-0.01425 -0.011312 -0.0006871"
       rpy="0 0 0" />
     <parent
-      link="camera_bottom_screw_frame" />
-    <child
-      link="camera_IMU_frame" />
+      link="camera_depth_frame" />
+    <child
+      link="camera_imu_frame" />
     <axis
       xyz="0 0 0" />
@@ -514,8 +514,8 @@
     type="fixed">
     <origin
-      xyz="0.0117149999999995 0.0475 0.0143111800025738"
+      xyz="0 0 0"
       rpy="0 0 0" />
     <parent
-      link="camera_bottom_screw_frame" />
+      link="camera_link" />
     <child
       link="camera_depth_frame" />

File: orbbec_description/urdf/test_astra2.urdf.xacro (robot description, xacro)
@@ -11,5 +11,5 @@
     <parent link="base_link"/>
     <child link="camera_link"/>
-    <origin xyz="0 0 0" rpy="0 0 0"/>
+    <origin xyz="0.012323996052145958 0.03750000149011612 0.028150320053100586" rpy="0 0 0"/>
   </joint>
 </robot>

File: orbbec_description/urdf/test_gemini2.urdf.xacro (robot description, xacro)
@@ -11,5 +11,5 @@
     <parent link="base_link"/>
     <child link="camera_link"/>
-    <origin xyz="0 0 0" rpy="0 0 0"/>
+    <origin xyz="0.01491 0.025 0.0125" rpy="0 0 0"/>
   </joint>
 </robot>

File: orbbec_description/urdf/test_gemini2L.urdf.xacro (robot description, xacro)
@@ -11,5 +11,5 @@
     <parent link="base_link"/>
     <child link="camera_link"/>
-    <origin xyz="0 0 0" rpy="0 0 0"/>
+    <origin xyz="0.01033 0.05 0.0145" rpy="0 0 0"/>
   </joint>
 </robot>

File: orbbec_description/urdf/test_gemini335L.urdf.xacro (robot description, xacro)
@@ -11,5 +11,5 @@
     <parent link="base_link"/>
     <child link="camera_link"/>
-    <origin xyz="0 0 0" rpy="0 0 0"/>
+    <origin xyz="0.011715 0.0475 0.014311" rpy="0 0 0"/>
   </joint>
 </robot>

File: orbbec_description/urdf/test_gemini335Le.urdf.xacro (robot description, xacro)
@@ -10,6 +10,6 @@
   <joint name="base_link_to_camera_link" type="fixed">
     <parent link="base_link"/>
-    <child link="camera_botton_screw_frame"/>
-    <origin xyz="0 0 0" rpy="0 0 0"/>
+    <child link="camera_link"/>
+    <origin xyz="0.034005 0.0475 0.014048" rpy="0 0 0"/>
   </joint>
 </robot>

File: orbbec_description/urdf/test_gemini335Lg.urdf.xacro (robot description, xacro)
@@ -11,5 +11,5 @@
     <parent link="base_link"/>
     <child link="camera_link"/>
-    <origin xyz="0 0 0" rpy="0 0 0"/>
+    <origin xyz="0.0117149999999995 0.0475 0.0143111800025738" rpy="0 0 0"/>
   </joint>
 </robot>

File: orbbec_description/urdf/test_gemini336L.urdf.xacro (robot description, xacro)
@@ -11,5 +11,5 @@
     <parent link="base_link"/>
     <child link="camera_link"/>
-    <origin xyz="0 0 0" rpy="0 0 0"/>
+    <origin xyz="0.011715 0.0475 0.014311" rpy="0 0 0"/>
   </joint>
 </robot>
